File: LED_Alarm.sch (KiCad schematic (older format))
At the start: 12 parts, among them U101 H11AA11, U102 ESP-12, U103 PCA9685PW

Commit message: After changes suggested in https://www.reddit.com/r/PrintedCircuitBoard/comments/54ctxv/pcb_review_of_a_pwm_esp8266_led_driver_board/
Parts:
- added P?: CONN_01X06, symbol CONN_01X06
- U102: footprint ESP8266:ESP-12 -> ESP8266:ESP-12E; symbol ESP-12 -> ESP-12E; Critical (none) -> No
Connections:
- net GNDREF: now also U102.15 (GND); no longer U102.9 (GND)
- net I2C_SDA: now also U102.17 (GPIO2); no longer U102.11 (GPIO2)
- net gpio0: now also U102.18 (GPIO0); no longer U102.12 (GPIO0)
- net gpio15: now also U102.16 (GPIO15); no longer U102.10 (GPIO15)
- net rx: now also U102.21 (RXD); no longer U102.15 (RXD)
- net tx: now also U102.22 (TXD); no longer U102.16 (TXD)
- net at U102.13 (MOSI): now also P?.2 (P2); no longer U103.23 (~OE)
- net at U102.14 (SCLK): now also P?.1 (P1)
- new net: P?.5 (P5), U102.10 (MISO)
- new net: P?.4 (P4), U102.11 (GPIO9)
- new net: P?.3 (P3), U102.12 (GPIO10)
- new net: U102.19 (GPIO4), U103.23 (~OE)
- new net: P?.6 (P6), U102.9 (CS0)
Other:
- moved on the sheet: C101
Changed lines of the file:
@@
 $EndDescr
 $Comp
-L ESP-12 U102
+L ESP-12E U102
 U 1 1 57DB3BB3
 P 3000 3600
 F 0 "U102" H 3000 3500 50  0000 C CNN
 F 1 "ESP-12" H 3000 3700 50  0000 C CNN
-F 2 "ESP8266:ESP-12" H 3000 3600 50  0001 C CNN
+F 2 "ESP8266:ESP-12E" H 3000 3600 50  0001 C CNN
 F 3 "" H 3000 3600 50  0001 C CNN
+F 4 "No" H 3000 3600 60  0001 C CNN "Critical"
 	1    3000 3600
 	1    0    0    -1
@@
 Text Label 1600 3800 0    60   ~ 0
 AC_CTRL1
-Text Label 2800 5250 2    60   ~ 0
+Text Label 2800 5600 2    60   ~ 0
 AC_CTRL1
 $Comp
@@
 $EndComp
 $Sheet
-S 2800 4900 700  800
+S 2800 5250 700  800
 U 57DD8455
 F0 "AC_Dimmer" 60
 F1 "AC_Dimmer.sch" 60
-F2 "AC_Control" I L 2800 5250 60
-$EndSheet
-$Sheet
-S 2800 6000 700  800
+F2 "AC_Control" I L 2800 5600 60
+$EndSheet
+$Sheet
+S 2800 6350 700  800
 U 57DD8BF5
 F0 "AC_Switch" 60
 F1 "AC_Switch.sch" 60
-F2 "AC_Control" I L 2800 6200 60
+F2 "AC_Control" I L 2800 6550 60
 $EndSheet
 Text Label 1600 3900 0    60   ~ 0
 AC_CTRL2
-Text Label 2800 6200 2    60   ~ 0
+Text Label 2800 6550 2    60   ~ 0
 AC_CTRL2
 Text Label 4950 3750 2    60   ~ 0
@@
 L GNDREF #PWR09
 U 1 1 57DD9951
-P 3000 4550
-F 0 "#PWR09" H 3000 4300 50  0001 C CNN
-F 1 "GNDREF" H 3000 4400 50  0000 C CNN
-F 2 "" H 3000 4550 50  0000 C CNN
-F 3 "" H 3000 4550 50  0000 C CNN
-	1    3000 4550
+P 3950 4000
+F 0 "#PWR09" H 3950 3750 50  0001 C CNN
+F 1 "GNDREF" H 3950 3850 50  0000 C CNN
+F 2 "" H 3950 4000 50  0000 C CNN
+F 3 "" H 3950 4000 50  0000 C CNN
+	1    3950 4000
 	1    0    0    -1
 $EndComp
@@
 L +3.3V #PWR010
 U 1 1 57DD99AD
-P 3000 2600
-F 0 "#PWR010" H 3000 2450 50  0001 C CNN
-F 1 "+3.3V" H 3000 2740 50  0000 C CNN
-F 2 "" H 3000 2600 50  0000 C CNN
-F 3 "" H 3000 2600 50  0000 C CNN
-	1    3000 2600
-	1    0    0    -1
+P 1900 4000
+F 0 "#PWR010" H 1900 3850 50  0001 C CNN
+F 1 "+3.3V" H 1900 4140 50  0000 C CNN
+F 2 "" H 1900 4000 50  0000 C CNN
+F 3 "" H 1900 4000 50  0000 C CNN
+	1    1900 4000
+	0    -1   -1   0
 $EndComp
 $Comp
@@
 L C_Small C101
 U 1 1 57DE57BD
-P 3150 2800
-F 0 "C101" H 3160 2870 50  0000 L CNN
-F 1 "C_Small" H 3160 2720 50  0000 L CNN
-F 2 "Capacitors_SMD:C_0603_HandSoldering" H 3150 2800 50  0001 C CNN
-F 3 "" H 3150 2800 50  0000 C CNN
-	1    3150 2800
+P 2000 4150
+F 0 "C101" H 2010 4220 50  0000 L CNN
+F 1 "C_Small" H 2010 4070 50  0000 L CNN
+F 2 "Capacitors_SMD:C_0603_HandSoldering" H 2000 4150 50  0001 C CNN
+F 3 "" H 2000 4150 50  0000 C CNN
+	1    2000 4150
 	1    0    0    -1
 $EndComp
@@
 	5050 3550 4450 3550
 Wire Wire Line
-	3000 4550 3000 4500
-Wire Wire Line
-	3000 2600 3000 2700
-Wire Wire Line
 	5850 2250 5850 2550
 Wire Wire Line
@@
 Wire Wire Line
 	4950 3350 5050 3350
-Wire Wire Line
-	3150 2700 3150 2650
-Wire Wire Line
-	3150 2650 3000 2650
-Connection ~ 3000 2650
 $Comp
 L GNDREF #PWR016
 U 1 1 57DE5F16
-P 3200 2900
-F 0 "#PWR016" H 3200 2650 50  0001 C CNN
-F 1 "GNDREF" H 3250 2550 50  0000 C CNN
-F 2 "" H 3200 2900 50  0000 C CNN
-F 3 "" H 3200 2900 50  0000 C CNN
-	1    3200 2900
-	0    -1   -1   0
-$EndComp
-Wire Wire Line
-	3200 2900 3150 2900
+P 2000 4350
+F 0 "#PWR016" H 2000 4100 50  0001 C CNN
+F 1 "GNDREF" H 2050 4000 50  0000 C CNN
+F 2 "" H 2000 4350 50  0000 C CNN
+F 3 "" H 2000 4350 50  0000 C CNN
+	1    2000 4350
+	1    0    0    -1
+$EndComp
 $Comp
 L GNDREF #PWR017
@@
 Wire Wire Line
 	4250 4700 4200 4700
+Wire Wire Line
+	3950 4000 3900 4000
+Wire Wire Line
+	1900 4000 2100 4000
+Wire Wire Line
+	2000 4000 2000 4050
+Connection ~ 2000 4000
+Wire Wire Line
+	2000 4350 2000 4250
+$Comp
+L CONN_01X06 P?
+U 1 1 57E78F15
+P 3000 4950
+F 0 "P?" V 2872 5278 50  0000 L CNN
+F 1 "CONN_01X06" V 2963 5278 50  0000 L CNN
+F 2 "" H 3000 4950 50  0000 C CNN
+F 3 "" H 3000 4950 50  0000 C CNN
+	1    3000 4950
+	0    1    1    0
+$EndComp
+Wire Wire Line
+	2750 4500 2750 4750
+Wire Wire Line
+	2850 4750 2850 4500
+Wire Wire Line
+	2950 4500 2950 4750
+Wire Wire Line
+	3050 4750 3050 4500
+Wire Wire Line
+	3150 4500 3150 4750
+Wire Wire Line
+	3250 4750 3250 4500
 $EndSCHEMATC

Commit message: changed some stuff around
Parts:
- added F101: PRG18BB101MB1RB, Resistors_SMD:R_0603_HandSoldering, symbol F_Small
- added VR101: MOV-07D221K-ND, Varistors:RV_Disc_D9_W3.5_P5, symbol VR
- P101: renamed from P?; footprint (none) -> Pin_Headers:Pin_Header_Straight_1x06
Connections:
- net GNDPWR: now also VR101.2
- net HT: now also VR101.1
- net at U101.1: now also F101.1; no longer R101.2
- new net: F101.2, R101.2
Other:
- moved on the sheet: R101
Changed lines of the file:
@@
 $EndComp
 $Comp
-L GNDREF #PWR01
+L GNDREF #PWR105
 U 1 1 57DB3CE6
 P 1200 1600
-F 0 "#PWR01" H 1200 1350 50  0001 C CNN
+F 0 "#PWR105" H 1200 1350 50  0001 C CNN
 F 1 "GNDREF" H 1200 1450 50  0000 C CNN
 F 2 "" H 1200 1600 50  0000 C CNN
@@
 ZX
 $Comp
-L GNDREF #PWR02
+L GNDREF #PWR109
 U 1 1 57DD719B
 P 1850 5550
-F 0 "#PWR02" H 1850 5300 50  0001 C CNN
+F 0 "#PWR109" H 1850 5300 50  0001 C CNN
 F 1 "GNDREF" H 1850 5400 50  0000 C CNN
 F 2 "" H 1850 5550 50  0000 C CNN
@@
 $EndComp
 $Comp
-L +3.3V #PWR03
+L +3.3V #PWR111
 U 1 1 57DD7221
 P 1900 5150
-F 0 "#PWR03" H 1900 5000 50  0001 C CNN
+F 0 "#PWR111" H 1900 5000 50  0001 C CNN
 F 1 "+3.3V" H 1900 5290 50  0000 C CNN
 F 2 "" H 1900 5150 50  0000 C CNN
@@
 L R_Small R101
 U 1 1 57DD72CB
-P 1100 5250
-F 0 "R101" H 1130 5270 50  0000 L CNN
-F 1 "68k" H 1130 5210 50  0000 L CNN
-F 2 "Resistors_ThroughHole:Resistor_Horizontal_RM10mm" H 1100 5250 50  0001 C CNN
-F 3 "" H 1100 5250 50  0000 C CNN
-	1    1100 5250
+P 1100 4800
+F 0 "R101" H 1130 4820 50  0000 L CNN
+F 1 "68k" H 1130 4760 50  0000 L CNN
+F 2 "Resistors_ThroughHole:Resistor_Horizontal_RM10mm" H 1100 4800 50  0001 C CNN
+F 3 "" H 1100 4800 50  0000 C CNN
+	1    1100 4800
 	1    0    0    -1
 $EndComp
@@
 AC_CTRL1
 $Comp
-L +12V #PWR04
+L +12V #PWR104
 U 1 1 57DD7FFF
 P 1200 1400
-F 0 "#PWR04" H 1200 1250 50  0001 C CNN
+F 0 "#PWR104" H 1200 1250 50  0001 C CNN
 F 1 "+12V" H 1200 1540 50  0000 C CNN
 F 2 "" H 1200 1400 50  0000 C CNN
@@
 $EndComp
 $Comp
-L HT #PWR05
-U 1 1 57DD813B
-P 1250 800
-F 0 "#PWR05" H 1250 920 50  0001 C CNN
-F 1 "HT" H 1250 890 50  0000 C CNN
-F 2 "" H 1250 800 50  0000 C CNN
-F 3 "" H 1250 800 50  0000 C CNN
-	1    1250 800
-	1    0    0    -1
-$EndComp
-$Comp
-L GNDPWR #PWR06
+L GNDPWR #PWR107
 U 1 1 57DD818F
 P 1250 1000
-F 0 "#PWR06" H 1250 800 50  0001 C CNN
+F 0 "#PWR107" H 1250 800 50  0001 C CNN
 F 1 "GNDPWR" H 1250 870 50  0000 C CNN
 F 2 "" H 1250 950 50  0000 C CNN
@@
 $EndComp
 $Comp
-L HT #PWR07
+L HT #PWR103
 U 1 1 57DD8276
-P 1100 5050
-F 0 "#PWR07" H 1100 5170 50  0001 C CNN
-F 1 "HT" H 1100 5140 50  0000 C CNN
-F 2 "" H 1100 5050 50  0000 C CNN
-F 3 "" H 1100 5050 50  0000 C CNN
-	1    1100 5050
-	1    0    0    -1
-$EndComp
-$Comp
-L GNDPWR #PWR08
+P 1100 4600
+F 0 "#PWR103" H 1100 4720 50  0001 C CNN
+F 1 "HT" H 1100 4690 50  0000 C CNN
+F 2 "" H 1100 4600 50  0000 C CNN
+F 3 "" H 1100 4600 50  0000 C CNN
+	1    1100 4600
+	1    0    0    -1
+$EndComp
+$Comp
+L GNDPWR #PWR102
 U 1 1 57DD82B1
-P 1050 5550
-F 0 "#PWR08" H 1050 5350 50  0001 C CNN
-F 1 "GNDPWR" H 1050 5420 50  0000 C CNN
-F 2 "" H 1050 5500 50  0000 C CNN
-F 3 "" H 1050 5500 50  0000 C CNN
-	1    1050 5550
+P 1000 5800
+F 0 "#PWR102" H 1000 5600 50  0001 C CNN
+F 1 "GNDPWR" H 1000 5670 50  0000 C CNN
+F 2 "" H 1000 5750 50  0000 C CNN
+F 3 "" H 1000 5750 50  0000 C CNN
+	1    1000 5800
 	1    0    0    -1
 $EndComp
@@
 I2C_SCL
 $Comp
-L GNDREF #PWR09
+L GNDREF #PWR113
 U 1 1 57DD9951
 P 3950 4000
-F 0 "#PWR09" H 3950 3750 50  0001 C CNN
+F 0 "#PWR113" H 3950 3750 50  0001 C CNN
 F 1 "GNDREF" H 3950 3850 50  0000 C CNN
 F 2 "" H 3950 4000 50  0000 C CNN
@@
 $EndComp
 $Comp
-L +3.3V #PWR010
+L +3.3V #PWR110
 U 1 1 57DD99AD
 P 1900 4000
-F 0 "#PWR010" H 1900 3850 50  0001 C CNN
+F 0 "#PWR110" H 1900 3850 50  0001 C CNN
 F 1 "+3.3V" H 1900 4140 50  0000 C CNN
 F 2 "" H 1900 4000 50  0000 C CNN
@@
 $EndComp
 $Comp
-L +3.3V #PWR011
+L +3.3V #PWR117
 U 1 1 57DD9B0F
 P 5850 2250
-F 0 "#PWR011" H 5850 2100 50  0001 C CNN
+F 0 "#PWR117" H 5850 2100 50  0001 C CNN
 F 1 "+3.3V" H 5850 2390 50  0000 C CNN
 F 2 "" H 5850 2250 50  0000 C CNN
@@
 $EndComp
 $Comp
-L GNDREF #PWR012
+L GNDREF #PWR118
 U 1 1 57DD9B66
 P 5850 4750
-F 0 "#PWR012" H 5850 4500 50  0001 C CNN
+F 0 "#PWR118" H 5850 4500 50  0001 C CNN
 F 1 "GNDREF" H 5850 4600 50  0000 C CNN
 F 2 "" H 5850 4750 50  0000 C CNN
@@
 $EndComp
 $Comp
-L GNDREF #PWR013
+L GNDREF #PWR101
 U 1 1 57DE15E2
 P 900 3300
-F 0 "#PWR013" H 900 3050 50  0001 C CNN
+F 0 "#PWR101" H 900 3050 50  0001 C CNN
 F 1 "GNDREF" H 900 3150 50  0000 C CNN
 F 2 "" H 900 3300 50  0000 C CNN
@@
 $EndComp
 $Comp
-L +3.3V #PWR014
+L +3.3V #PWR108
 U 1 1 57DE1A8C
 P 1800 3000
-F 0 "#PWR014" H 1800 2850 50  0001 C CNN
+F 0 "#PWR108" H 1800 2850 50  0001 C CNN
 F 1 "+3.3V" H 1800 3140 50  0000 C CNN
 F 2 "" H 1800 3000 50  0000 C CNN
@@
 rx
 $Comp
-L GNDREF #PWR015
+L GNDREF #PWR115
 U 1 1 57DE3EAE
 P 4650 2950
-F 0 "#PWR015" H 4650 2700 50  0001 C CNN
+F 0 "#PWR115" H 4650 2700 50  0001 C CNN
 F 1 "GNDREF" H 4650 2800 50  0000 C CNN
 F 2 "" H 4650 2950 50  0000 C CNN
@@
 $EndComp
 Wire Wire Line
-	1250 950  1150 950
-Wire Wire Line
-	1250 850  1150 850
+	1150 950  1450 950
+Wire Wire Line
+	1150 850  1450 850
 Wire Wire Line
 	1150 1550 1200 1550
@@
 	1900 5150 1900 5200
 Wire Wire Line
-	1050 5550 1200 5550
-Wire Wire Line
-	1100 5050 1100 5150
-Wire Wire Line
-	1100 5350 1200 5350
+	1000 5550 1200 5550
+Wire Wire Line
+	1100 4600 1100 4700
+Wire Wire Line
+	950  5350 1200 5350
 Wire Wire Line
 	1600 3700 2100 3700
@@
 	4950 3350 5050 3350
 $Comp
-L GNDREF #PWR016
+L GNDREF #PWR112
 U 1 1 57DE5F16
 P 2000 4350
-F 0 "#PWR016" H 2000 4100 50  0001 C CNN
+F 0 "#PWR112" H 2000 4100 50  0001 C CNN
 F 1 "GNDREF" H 2050 4000 50  0000 C CNN
 F 2 "" H 2000 4350 50  0000 C CNN
@@
 $EndComp
 $Comp
-L GNDREF #PWR017
+L GNDREF #PWR119
 U 1 1 57DE609D
 P 6250 2600
-F 0 "#PWR017" H 6250 2350 50  0001 C CNN
+F 0 "#PWR119" H 6250 2350 50  0001 C CNN
 F 1 "GNDREF" H 6250 2450 50  0000 C CNN
 F 2 "" H 6250 2600 50  0000 C CNN
@@
 	7050 2400 8300 2400
 $Comp
-L GNDREF #PWR018
+L GNDREF #PWR116
 U 1 1 57E4B837
 P 5000 4300
-F 0 "#PWR018" H 5000 4050 50  0001 C CNN
+F 0 "#PWR116" H 5000 4050 50  0001 C CNN
 F 1 "GNDREF" H 5000 4150 50  0000 C CNN
 F 2 "" H 5000 4300 50  0000 C CNN
@@
 $EndComp
 $Comp
-L +3.3V #PWR019
+L +3.3V #PWR114
 U 1 1 57E51206
 P 4500 4700
-F 0 "#PWR019" H 4500 4550 50  0001 C CNN
+F 0 "#PWR114" H 4500 4550 50  0001 C CNN
 F 1 "+3.3V" H 4500 4840 50  0000 C CNN
 F 2 "" H 4500 4700 50  0000 C CNN
@@
 	2000 4350 2000 4250
 $Comp
-L CONN_01X06 P?
+L CONN_01X06 P101
 U 1 1 57E78F15
 P 3000 4950
-F 0 "P?" V 2872 5278 50  0000 L CNN
-F 1 "CONN_01X06" V 2963 5278 50  0000 L CNN
-F 2 "" H 3000 4950 50  0000 C CNN
+F 0 "P101" V 2827 5278 50  0000 L CNN
+F 1 "CONN_01X06" V 2918 5278 50  0000 L CNN
+F 2 "Pin_Headers:Pin_Header_Straight_1x06" V 3009 5278 50  0000 L CNN
 F 3 "" H 3000 4950 50  0000 C CNN
 	1    3000 4950
@@
 Wire Wire Line
 	3250 4750 3250 4500
+Wire Wire Line
+	1000 5550 1000 5800
+Wire Wire Line
+	1000 5700 800  5700
+Connection ~ 1000 5700
+Wire Wire Line
+	950  5350 950  5100
+Wire Wire Line
+	950  5100 800  5100
+Connection ~ 1100 5350
+$Comp
+L VR VR101
+U 1 1 57EB18A3
+P 1600 950
+F 0 "VR101" V 1660 904 50  0000 C TNN
+F 1 "MOV-07D221K-ND" V 1600 950 50  0000 C CNN
+F 2 "Varistors:RV_Disc_D9_W3.5_P5" H 1600 950 50  0001 C CNN
+F 3 "" H 1600 950 50  0000 C CNN
+	1    1600 950
+	1    0    0    -1
+$EndComp
+Wire Wire Line
+	1600 700  1450 700
+Wire Wire Line
+	1450 700  1450 850
+Connection ~ 1250 850
+Wire Wire Line
+	1450 950  1450 1200
+Wire Wire Line
+	1450 1200 1600 1200
+Connection ~ 1250 950
+$Comp
+L HT #PWR106
+U 1 1 57DD813B
+P 1250 800
+F 0 "#PWR106" H 1250 920 50  0001 C CNN
+F 1 "HT" H 1250 890 50  0000 C CNN
+F 2 "" H 1250 800 50  0000 C CNN
+F 3 "" H 1250 800 50  0000 C CNN
+	1    1250 800
+	1    0    0    -1
+$EndComp
+$Comp
+L F_Small F101
+U 1 1 57EB2669
+P 1100 5150
+F 0 "F101" H 1060 5210 50  0000 L CNN
+F 1 "PRG18BB101MB1RB" H 980 5090 50  0000 L CNN
+F 2 "Resistors_SMD:R_0603_HandSoldering" H 1100 5150 50  0001 C CNN
+F 3 "" H 1100 5150 50  0000 C CNN
+	1    1100 5150
+	0    -1   -1   0
+$EndComp
+Wire Wire Line
+	1100 4900 1100 5050
+Wire Wire Line
+	1100 5250 1100 5350
 $EndSCHEMATC
