File: LED_Control.sch (KiCad schematic (older format))
At the start: 7 parts, among them Q401 FDMA410NZT, Q402 FDMA410NZT, Q403 FDMA410NZT

Commit message: changed some stuff around
Parts:
- C401: footprint Capacitors_SMD:c_elec_10x10 -> HouseFootprints:c_elec_8.3x8.3
Changed lines of the file:
@@
 AR Path="/57DDA0A5/57DD9DC5" Ref="Q701"  Part="1"
 AR Path="/57DDACE8/57DD9DC5" Ref="Q801"  Part="1"
-F 0 "Q401" H 2100 1800 50  0000 R CNN
+F 0 "Q501" H 2100 1800 50  0000 R CNN
 F 1 "FDMA410NZT" H 2450 1700 50  0000 R CNN
 F 2 "HouseFootprints:MicroFET-6" H 2000 1850 50  0001 C CNN
@@
 AR Path="/57DDA0A5/57DD9DEF" Ref="#PWR051"  Part="1"
 AR Path="/57DDACE8/57DD9DEF" Ref="#PWR059"  Part="1"
-F 0 "#PWR027" H 1900 1750 50  0001 C CNN
+F 0 "#PWR035" H 1900 1750 50  0001 C CNN
 F 1 "GNDREF" H 1900 1850 50  0000 C CNN
 F 2 "" H 1900 2000 50  0000 C CNN
@@
 AR Path="/57DDA0A5/57DD9E09" Ref="LED0"  Part="1"
 AR Path="/57DDACE8/57DD9E09" Ref="LED5"  Part="1"
-F 0 "LED9" H 2100 1350 50  0000 C CNN
+F 0 "LED3" H 2100 1350 50  0000 C CNN
 F 1 "CONN_01X02" V 2200 1200 50  0000 C CNN
 F 2 "Pin_Headers:Pin_Header_Straight_1x02" H 2100 1200 50  0001 C CNN
@@
 AR Path="/57DDA0A5/57DD9E42" Ref="#PWR052"  Part="1"
 AR Path="/57DDACE8/57DD9E42" Ref="#PWR060"  Part="1"
-F 0 "#PWR028" H 1900 950 50  0001 C CNN
+F 0 "#PWR036" H 1900 950 50  0001 C CNN
 F 1 "+12V" H 1900 1240 50  0000 C CNN
 F 2 "" H 1900 1100 50  0000 C CNN
@@
 AR Path="/57DDA0A5/57DDA2C6" Ref="LED1"  Part="1"
 AR Path="/57DDACE8/57DDA2C6" Ref="LED6"  Part="1"
-F 0 "LED10" H 2100 2650 50  0000 C CNN
+F 0 "LED4" H 2100 2650 50  0000 C CNN
 F 1 "CONN_01X02" V 2300 2500 50  0000 C CNN
 F 2 "Pin_Headers:Pin_Header_Straight_1x02" H 2100 2500 50  0001 C CNN
@@
 AR Path="/57DDA0A5/57DDA2CD" Ref="#PWR053"  Part="1"
 AR Path="/57DDACE8/57DDA2CD" Ref="#PWR061"  Part="1"
-F 0 "#PWR029" H 1900 2250 50  0001 C CNN
+F 0 "#PWR037" H 1900 2250 50  0001 C CNN
 F 1 "+12V" H 1900 2540 50  0000 C CNN
 F 2 "" H 1900 2400 50  0000 C CNN
@@
 AR Path="/57DDA0A5/57DDA338" Ref="#PWR054"  Part="1"
 AR Path="/57DDACE8/57DDA338" Ref="#PWR062"  Part="1"
-F 0 "#PWR030" H 1900 4550 50  0001 C CNN
+F 0 "#PWR038" H 1900 4550 50  0001 C CNN
 F 1 "GNDREF" H 1900 4650 50  0000 C CNN
 F 2 "" H 1900 4800 50  0000 C CNN
@@
 AR Path="/57DDA0A5/57DDA33F" Ref="LED2"  Part="1"
 AR Path="/57DDACE8/57DDA33F" Ref="LED8"  Part="1"
-F 0 "LED11" H 2100 4150 50  0000 C CNN
+F 0 "LED7" H 2100 4150 50  0000 C CNN
 F 1 "CONN_01X02" V 2400 4000 50  0000 C CNN
 F 2 "Pin_Headers:Pin_Header_Straight_1x02" H 2100 4000 50  0001 C CNN
@@
 AR Path="/57DDA0A5/57DDA346" Ref="#PWR055"  Part="1"
 AR Path="/57DDACE8/57DDA346" Ref="#PWR063"  Part="1"
-F 0 "#PWR031" H 1900 3750 50  0001 C CNN
+F 0 "#PWR039" H 1900 3750 50  0001 C CNN
 F 1 "+12V" H 1900 4040 50  0000 C CNN
 F 2 "" H 1900 3900 50  0000 C CNN
@@
 AR Path="/57DDA0A5/57DDA2BF" Ref="#PWR056"  Part="1"
 AR Path="/57DDACE8/57DDA2BF" Ref="#PWR064"  Part="1"
-F 0 "#PWR032" H 1900 3050 50  0001 C CNN
+F 0 "#PWR040" H 1900 3050 50  0001 C CNN
 F 1 "GNDREF" H 1900 3150 50  0000 C CNN
 F 2 "" H 1900 3300 50  0000 C CNN
@@
 AR Path="/57DDA0A5/57DECFD1" Ref="Q702"  Part="1"
 AR Path="/57DDACE8/57DECFD1" Ref="Q802"  Part="1"
-F 0 "Q402" H 2100 3100 50  0000 R CNN
+F 0 "Q502" H 2100 3100 50  0000 R CNN
 F 1 "FDMA410NZT" H 2450 3000 50  0000 R CNN
 F 2 "HouseFootprints:MicroFET-6" H 2000 3150 50  0001 C CNN
@@
 AR Path="/57DDA0A5/57DECFFA" Ref="Q703"  Part="1"
 AR Path="/57DDACE8/57DECFFA" Ref="Q803"  Part="1"
-F 0 "Q403" H 2100 4600 50  0000 R CNN
+F 0 "Q503" H 2100 4600 50  0000 R CNN
 F 1 "FDMA410NZT" H 2450 4500 50  0000 R CNN
 F 2 "HouseFootprints:MicroFET-6" H 2000 4650 50  0001 C CNN
@@
 AR Path="/57DDA0A5/57E53674" Ref="C701"  Part="1"
 AR Path="/57DDACE8/57E53674" Ref="C801"  Part="1"
-F 0 "C401" H 3115 1591 50  0000 L CNN
+F 0 "C501" H 3115 1591 50  0000 L CNN
 F 1 "CP1" H 3115 1500 50  0000 L CNN
-F 2 "Capacitors_SMD:c_elec_10x10" H 3115 1409 50  0000 L CNN
+F 2 "HouseFootprints:c_elec_8.3x8.3" H 3115 1409 50  0000 L CNN
 F 3 "" H 3000 1500 50  0000 C CNN
 	1    3000 1500
@@
 AR Path="/57DDA0A5/57E536D5" Ref="#PWR057"  Part="1"
 AR Path="/57DDACE8/57E536D5" Ref="#PWR065"  Part="1"
-F 0 "#PWR033" H 3000 1150 50  0001 C CNN
+F 0 "#PWR041" H 3000 1150 50  0001 C CNN
 F 1 "+12V" H 3000 1440 50  0000 C CNN
 F 2 "" H 3000 1300 50  0000 C CNN
@@
 AR Path="/57DDA0A5/57E536FE" Ref="#PWR058"  Part="1"
 AR Path="/57DDACE8/57E536FE" Ref="#PWR066"  Part="1"
-F 0 "#PWR034" H 3000 1450 50  0001 C CNN
+F 0 "#PWR042" H 3000 1450 50  0001 C CNN
 F 1 "GNDREF" H 3000 1550 50  0000 C CNN
 F 2 "" H 3000 1700 50  0000 C CNN
