File: Programmer.sch (KiCad schematic (older format))
At the start: 11 parts

Commit message: changed some stuff around
Connections:
- net +3V3: now also FTDI1001.3 (P3)
Changed lines of the file:
@@
 	1    0    0    -1
 $EndComp
+$Comp
+L +3.3V #PWR081
+U 1 1 57E79D66
+P 4250 3100
+F 0 "#PWR081" H 4250 2950 50  0001 C CNN
+F 1 "+3.3V" H 4250 3240 50  0000 C CNN
+F 2 "" H 4250 3100 50  0000 C CNN
+F 3 "" H 4250 3100 50  0000 C CNN
+	1    4250 3100
+	1    0    0    -1
+$EndComp
+Wire Wire Line
+	4250 3100 4550 3100
 $EndSCHEMATC
